Commit message: alteração no arquivo domain.xacro

File: urdf/domain.xacro (robot description, xacro)
@@ -1,440 +1,128 @@
-<?xml version="1.0" encoding="utf-8"?>
-<!--
-  Model primitives.
-  Author: Helio Perroni Filho
--->
-<robot xmlns:xacro="http://www.ros.org/wiki/xacro">
-  <!-- Predefined constants. -->
-  <xacro:property name="M_PI" value="${pi}"/>
-  <xacro:property name="M_PI_2" value="${0.5 * M_PI}"/>
-  <xacro:property name="DEG" value="${M_PI / 180.0}"/>
-  <!-- Default density for computing object mass based on volume. -->
-  <xacro:property name="DENSITY" value="200.0"/>
-  <!-- Pre-defined material colors. -->
-  <material name="Black">
-    <color rgba="0.0 0.0 0.0 1.0"/>
-  </material>
-  <material name="White">
-    <color rgba="1.0 1.0 1.0 1.0"/>
-  </material>
-  <material name="Grey">
-    <color rgba="0.3 0.3 0.3 1.0"/>
-  </material>
-  <material name="DarkGrey">
-    <color rgba="0.175 0.175 0.175 1.0"/>
-  </material>
-  <!-- Placeholder inertial tensor. -->
-  <xacro:macro
-    name="inertia_none"
-  >
-    <inertia
-      ixx="0.0" ixy="0.0"  ixz="0.0"
-      iyy="0.0" iyz="0.0"
-      izz="0.0"
-    />
-  </xacro:macro>
-  <!-- Compute the inertial tensor of a block. -->
-  <xacro:macro
-    name="inertia_block"
-    params="
-      mass
-      size_x
-      size_y
-      size_z
-    "
-  >
-    <inertia
-      ixx="${mass * (size_z ** 2.0 + size_y ** 2.0) / 12.0}" ixy="0.0"  ixz="0.0"
-      iyy="${mass * (size_x ** 2.0 + size_z ** 2.0) / 12.0}" iyz="0.0"
-      izz="${mass * (size_x ** 2.0 + size_y ** 2.0) / 12.0}"
-    />
-  </xacro:macro>
-  <!-- Compute the inertial tensor of a cylinder. -->
-  <xacro:macro
-    name="inertia_cylinder"
-    params="
-      mass
-      radius
-      length
-    "
-  >
-    <inertia
-      ixx="${mass * (3.0 * radius ** 2.0 + length ** 2.0) / 12.0}" ixy="0.0"  ixz="0.0"
-      iyy="${mass * (3.0 * radius ** 2.0 + length ** 2.0) / 12.0}" iyz="0.0"
-      izz="${0.5 * mass * radius ** 2.0}"
-    />
-  </xacro:macro>
-  <!-- Compute the inertial tensor of a sphere. -->
-  <xacro:macro
-    name="inertia_sphere"
-    params="
-      mass
-      radius
-    "
-  >
-    <inertia
-      ixx="${0.4 * mass * radius ** 2.0}" ixy="0.0"  ixz="0.0"
-      iyy="${0.4 * mass * radius ** 2.0}" iyz="0.0"
-      izz="${0.4 * mass * radius ** 2.0}"
-    />
-  </xacro:macro>
-  <!-- Create a solid of given parameters. -->
-  <xacro:macro
-    name="solid_object"
-    params="
-      name
-      x:=0.0
-      y:=0.0
-      z:=0.0
-      roll:=0.0
-      pitch:=0.0
-      yaw:=0.0
-      mass:=0.0
-      material:=''
-      visible:=true
-      *inertia
-      *geometry
-    "
-  >
-    <link name="${name}">
-      <xacro:if value="${mass > 0.0}">
-        <inertial>
-          <origin xyz="${x} ${y} ${z}" rpy="${roll} ${pitch} ${yaw}"/>
-          <mass value="${mass}"/>
-          <xacro:insert_block name="inertia"/>
-        </inertial>
-      </xacro:if>
-      <xacro:if value="${visible}">
-        <visual>
-          <origin xyz="${x} ${y} ${z}" rpy="${roll} ${pitch} ${yaw}"/>
-          <geometry>
-            <xacro:insert_block name="geometry"/>
-          </geometry>
-          <xacro:if value="${material != ''}">
-            <material name="${material}"/>
-          </xacro:if>
-        </visual>
-      </xacro:if>
-      <xacro:if value="${mass > 0.0}">
-        <collision>
-          <origin xyz="${x} ${y} ${z}" rpy="${roll} ${pitch} ${yaw}"/>
-          <geometry>
-            <xacro:insert_block name="geometry"/>
-          </geometry>
-        </collision>
-      </xacro:if>
-    </link>
-    <xacro:if value="${material != ''}">
-      <gazebo reference="${name}">
-        <material>Gazebo/${material}</material>
-      </gazebo>
-    </xacro:if>
-  </xacro:macro>
-  <!-- Create a solid cuboid block of given parameters. -->
-  <xacro:macro
-    name="solid_block"
-    params="
-      name
-      x:=0.0
-      y:=0.0
-      z:=0.0
-      roll:=0.0
-      pitch:=0.0
-      yaw:=0.0
-      size_x:=1.0
-      size_y:=1.0
-      size_z:=1.0
-      mass:=-1.0
-      material:='Grey'
-      visible:=true
-    "
-  >
-    <xacro:property name="mass_block" value="${mass if mass >= 0.0 else DENSITY * size_x * size_y * size_z}"/>
-    <xacro:solid_object
-      name="${name}"
-      x="${x}"
-      y="${y}"
-      z="${z}"
-      roll="${roll}"
-      pitch="${pitch}"
-      yaw="${yaw}"
-      mass="${mass_block}"
-      material="${material}"
-      visible="${visible}"
-    >
-      <xacro:inertia_block
-        mass="${mass_block}"
-        size_x="${size_x}"
-        size_y="${size_y}"
-        size_z="${size_z}"
-      />
-      <box size="${size_x} ${size_y} ${size_z}"/>
-    </xacro:solid_object>
-  </xacro:macro>
-  <!-- Create a solid cylinder of given parameters. -->
-  <xacro:macro
-    name="solid_cylinder"
-    params="
-      name
-      x:=0.0
-      y:=0.0
-      z:=0.0
-      roll:=0.0
-      pitch:=0.0
-      yaw:=0.0
-      radius:=0.5
-      length:=1.0
-      mass:=-1.0
-      material:='Grey'
-      visible:=true
-    "
-  >
-    <xacro:property name="mass_cylinder" value="${mass if mass >= 0.0 else DENSITY * length * pi * radius ** 2.0}"/>
-    <xacro:solid_object
-      name="${name}"
-      x="${x}"
-      y="${y}"
-      z="${z}"
-      roll="${roll}"
-      pitch="${pitch}"
-      yaw="${yaw}"
-      mass="${mass_cylinder}"
-      material="${material}"
-      visible="${visible}"
-    >
-      <xacro:inertia_cylinder
-        mass="${mass_cylinder}"
-        radius="${radius}"
-        length="${length}"
-      />
-      <cylinder radius="${radius}" length="${length}"/>
-    </xacro:solid_object>
-  </xacro:macro>
-  <!-- Create a solid sphere of given parameters. -->
-  <xacro:macro
-    name="solid_sphere"
-    params="
-      name
-      x:=0.0
-      y:=0.0
-      z:=0.0
-      roll:=0.0
-      pitch:=0.0
-      yaw:=0.0
-      radius:=0.5
-      mass:=-1.0
-      material:='Grey'
-      visible:=true
-    "
-  >
-    <xacro:property name="mass_sphere" value="${mass if mass >= 0.0 else DENSITY * 1.33 * pi * radius ** 2.0}"/>
-    <xacro:solid_object
-      name="${name}"
-      x="${x}"
-      y="${y}"
-      z="${z}"
-      roll="${roll}"
-      pitch="${pitch}"
-      yaw="${yaw}"
-      mass="${mass_sphere}"
-      material="${material}"
-      visible="${visible}"
-    >
-      <xacro:inertia_sphere
-        mass="${mass_sphere}"
-        radius="${radius}"
-      />
-      <sphere radius="${radius}"/>
-    </xacro:solid_object>
-  </xacro:macro>
+<?xml version="1.0"?>
+<robot xmlns:xacro="http://www.ros.org/wiki/xacro" name="rosbot3">
   <!--
-    Create a mesh of given parameters.
-    The filename parameter is a URL, therefore local files should be prepended by
-    "file://", for example:
-    <xacro:solid_mesh name="link_name" filename="file://$(find package_name)/urdf/mesh.stl">
-      ...
-    </xacro:solid_mesh>
+    Este arquivo assume que o seu domain.xacro (o arquivo que você mostrou)
+    está em: $(find my_robot_description)/urdf/domain.xacro
+    Ajuste o caminho abaixo conforme seu pacote.
   -->
-  <xacro:macro
-    name="solid_mesh"
-    params="
-      name
-      filename
-      scale:=1.0
-      x:=0.0
-      y:=0.0
-      z:=0.0
-      roll:=0.0
-      pitch:=0.0
-      yaw:=0.0
-      mass:=0.0
-      material:=''
-      visible:=true
-      *inertia
-    "
-  >
-    <xacro:solid_object
-      name="${name}"
-      x="${x}"
-      y="${y}"
-      z="${z}"
-      roll="${roll}"
-      pitch="${pitch}"
-      yaw="${yaw}"
-      mass="${mass}"
-      material="${material}"
-      visible="${visible}"
-    >
-      <xacro:insert_block name="inertia"/>
-      <mesh filename="${filename}" scale="${scale} ${scale} ${scale}"/>
-    </xacro:solid_object>
-  </xacro:macro>
-  <!-- Create a joint of given type between two links. -->
-  <xacro:macro
-    name="joint_of"
-    params="
-      type
-      name:=''
-      parent
-      child
-      x:=0.0
-      y:=0.0
-      z:=0.0
-      roll:=0.0
-      pitch:=0.0
-      yaw:=0.0
-      **extensions
-    "
-  >
-    <joint name="${name if name != '' else 'joint_%s_%s' % (parent, child)}" type="${type}">
-      <parent link="${parent}"/>
-      <child link="${child}"/>
-      <origin xyz="${x} ${y} ${z}" rpy="${roll} ${pitch} ${yaw}"/>
-      <xacro:insert_block name="extensions"/>
-    </joint>
-  </xacro:macro>
-  <!-- Create a fixed joint between two links. -->
-  <xacro:macro
-    name="joint_fixed"
-    params="
-      name:=''
-      parent
-      child
-      x:=0.0
-      y:=0.0
-      z:=0.0
-      roll:=0.0
-      pitch:=0.0
-      yaw:=0.0
-    "
-  >
-    <xacro:joint_of type="fixed"
-      name="${name}"
-      parent="${parent}"
-      child="${child}"
-      x="${x}"
-      y="${y}"
-      z="${z}"
-      roll="${roll}"
-      pitch="${pitch}"
-      yaw="${yaw}"
-    >
-      <extensions/>
-    </xacro:joint_of>
-  </xacro:macro>
-  <!-- Create a continuous joint between two links. -->
-  <xacro:macro
-    name="joint_continuous"
-    params="
-      name:=''
-      parent
-      child
-      axis:='1 0 0'
-      x:=0.0
-      y:=0.0
-      z:=0.0
-      roll:=0.0
-      pitch:=0.0
-      yaw:=0.0
-    "
-  >
-    <xacro:joint_of type="continuous"
-      name="${name}"
-      parent="${parent}"
-      child="${child}"
-      x="${x}"
-      y="${y}"
-      z="${z}"
-      roll="${roll}"
-      pitch="${pitch}"
-      yaw="${yaw}"
-    >
-      <extensions>
-        <axis xyz="${axis}"/>
-      </extensions>
-    </xacro:joint_of>
-  </xacro:macro>
-  <!-- Create a joint effected by an actuator (real or simulated). -->
-  <xacro:macro
-    name="joint_actuated"
-    params="
-      name
-      parent
-      child
-      type:='revolute'
-      axis:='1 0 0'
-      effort:=10.0
-      velocity:=1.0
-      lower:=${-M_PI}
-      upper:=${M_PI}
-      x:=0.0
-      y:=0.0
-      z:=0.0
-      roll:=0.0
-      pitch:=0.0
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
Commit message: nova versão do ros_commons

File: urdf/domain.xacro (robot description, xacro)
@@ -1,128 +1,527 @@
-<?xml version="1.0"?>
-<robot xmlns:xacro="http://www.ros.org/wiki/xacro" name="rosbot3">
+<?xml version="1.0" encoding="utf-8"?>
+<!--
+  Model primitives.
+  Autor original: Helio Perroni Filho
+  Adaptado por: Vito Rodrigues Franzosi
+  Date: 06.11.2025
+-->
+<robot xmlns:xacro="http://www.ros.org/wiki/xacro">
+  <!-- Predefined constants. -->
+  <xacro:property name="M_PI" value="${pi}"/>
+  <xacro:property name="M_PI_2" value="${0.5 * M_PI}"/>
+  <xacro:property name="DEG" value="${M_PI / 180.0}"/>
+  <!-- Default density for computing object mass based on volume. -->
+  <xacro:property name="DENSITY" value="200.0"/>
+  <!-- Pre-defined material colors. -->
+  <material name="Black">
+    <color rgba="0.0 0.0 0.0 1.0"/>
+  </material>
+  <material name="White">
+    <color rgba="1.0 1.0 1.0 1.0"/>
+  </material>
+  <material name="Grey">
+    <color rgba="0.3 0.3 0.3 1.0"/>
+  </material>
+  <material name="DarkGrey">
+    <color rgba="0.175 0.175 0.175 1.0"/>
+  </material>
+  <material name="Red">
+    <color rgba="1.0 0.0 0.0 1.0"/>
+  </material>
+  <!-- Placeholder inertial tensor. -->
+  <xacro:macro
+    name="inertia_none"
+  >
+    <inertia
+      ixx="0.0" ixy="0.0"  ixz="0.0"
+      iyy="0.0" iyz="0.0"
+      izz="0.0"
+    />
+  </xacro:macro>
+  <!-- Compute the inertial tensor of a block. -->
+  <xacro:macro
+    name="inertia_block"
+    params="
+      mass
+      size_x
+      size_y
+      size_z
+    "
+  >
+    <inertia
+      ixx="${mass * (size_z ** 2.0 + size_y ** 2.0) / 12.0}" ixy="0.0"  ixz="0.0"
+      iyy="${mass * (size_x ** 2.0 + size_z ** 2.0) / 12.0}" iyz="0.0"
+      izz="${mass * (size_x ** 2.0 + size_y ** 2.0) / 12.0}"
+    />
+  </xacro:macro>
+  <!-- Compute the inertial tensor of a cylinder. -->
+  <xacro:macro
+    name="inertia_cylinder"
+    params="
+      mass
+      radius
+      length
+    "
+  >
+    <inertia
+      ixx="${mass * (3.0 * radius ** 2.0 + length ** 2.0) / 12.0}" ixy="0.0"  ixz="0.0"
+      iyy="${mass * (3.0 * radius ** 2.0 + length ** 2.0) / 12.0}" iyz="0.0"
+      izz="${0.5 * mass * radius ** 2.0}"
+    />
+  </xacro:macro>
+  <!-- Compute the inertial tensor of a sphere. -->
+  <xacro:macro
+    name="inertia_sphere"
+    params="
+      mass
+      radius
+    "
+  >
+    <inertia
+      ixx="${0.4 * mass * radius ** 2.0}" ixy="0.0"  ixz="0.0"
+      iyy="${0.4 * mass * radius ** 2.0}" iyz="0.0"
+      izz="${0.4 * mass * radius ** 2.0}"
+    />
+  </xacro:macro>
+  <!-- Create a solid of given parameters. -->
+  <xacro:macro
+    name="solid_object"
+    params="
+      name
+      x:=0.0
+      y:=0.0
+      z:=0.0
+      roll:=0.0
+      pitch:=0.0
+      yaw:=0.0
+      mass:=0.0
+      material:=''
+      visible:=true
+      *inertia
+      *geometry
+    "
+  >
+    <link name="${name}">
+      <xacro:if value="${mass > 0.0}">
+        <inertial>
+          <origin xyz="${x} ${y} ${z}" rpy="${roll} ${pitch} ${yaw}"/>
+          <mass value="${mass}"/>
+          <xacro:insert_block name="inertia"/>
+        </inertial>
+      </xacro:if>
+      <xacro:if value="${visible}">
+        <visual>
+          <origin xyz="${x} ${y} ${z}" rpy="${roll} ${pitch} ${yaw}"/>
+          <geometry>
+            <xacro:insert_block name="geometry"/>
+          </geometry>
+          <xacro:if value="${material != ''}">
+            <material name="${material}"/>
+          </xacro:if>
+        </visual>
+      </xacro:if>
+      <xacro:if value="${mass > 0.0}">
+        <collision>
+          <origin xyz="${x} ${y} ${z}" rpy="${roll} ${pitch} ${yaw}"/>
+          <geometry>
+            <xacro:insert_block name="geometry"/>
+          </geometry>
+        </collision>
+      </xacro:if>
+    </link>
+    <xacro:if value="${material != ''}">
+      <gazebo reference="${name}">
+        <material>Gazebo/${material}</material>
+      </gazebo>
+    </xacro:if>
+  </xacro:macro>
+  <!-- Create a solid cuboid block of given parameters. -->
+  <xacro:macro
+    name="solid_block"
+    params="
+      name
+      x:=0.0
+      y:=0.0
+      z:=0.0
+      roll:=0.0
+      pitch:=0.0
+      yaw:=0.0
+      size_x:=1.0
+      size_y:=1.0
+      size_z:=1.0
+      mass:=-1.0
+      material:='Grey'
+      visible:=true
+    "
+  >
+    <xacro:property name="mass_block" value="${mass if mass >= 0.0 else DENSITY * size_x * size_y * size_z}"/>
+    <xacro:solid_object
+      name="${name}"
+      x="${x}"
+      y="${y}"
+      z="${z}"
+      roll="${roll}"
+      pitch="${pitch}"
+      yaw="${yaw}"
+      mass="${mass_block}"
+      material="${material}"
+      visible="${visible}"
+    >
+      <xacro:inertia_block
+        mass="${mass_block}"
+        size_x="${size_x}"
+        size_y="${size_y}"
+        size_z="${size_z}"
+      />
+      <box size="${size_x} ${size_y} ${size_z}"/>
+    </xacro:solid_object>
+  </xacro:macro>
+  <!-- Create a solid cuboid block of given parameters. -->
+  <xacro:macro
+    name="solid_block_red"
+    params="
+      name
+      x:=0.0
+      y:=0.0
+      z:=0.0
+      roll:=0.0
+      pitch:=0.0
+      yaw:=0.0
+      size_x:=1.0
+      size_y:=1.0
+      size_z:=1.0
+      mass:=-1.0
+      material:='Red'
+      visible:=true
+    "
+  >
+    <xacro:property name="mass_block" value="${mass if mass >= 0.0 else DENSITY * size_x * size_y * size_z}"/>
+    <xacro:solid_object
+      name="${name}"
+      x="${x}"
+      y="${y}"
+      z="${z}"
+      roll="${roll}"
+      pitch="${pitch}"
+      yaw="${yaw}"
+      mass="${mass_block}"
+      material="${material}"
+      visible="${visible}"
+    >
+      <xacro:inertia_block
+        mass="${mass_block}"
+        size_x="${size_x}"
+        size_y="${size_y}"
+        size_z="${size_z}"
+      />
+      <box size="${size_x} ${size_y} ${size_z}"/>
+    </xacro:solid_object>
+  </xacro:macro>
+  <!-- Create a solid cuboid block of given parameters. -->
+  <xacro:macro
+    name="solid_block_black"
+    params="
+      name
+      x:=0.0
+      y:=0.0
+      z:=0.0
+      roll:=0.0
+      pitch:=0.0
+      yaw:=0.0
+      size_x:=1.0
+      size_y:=1.0
+      size_z:=1.0
+      mass:=-1.0
+      material:='Black'
+      visible:=true
+    "
+  >
+    <xacro:property name="mass_block" value="${mass if mass >= 0.0 else DENSITY * size_x * size_y * size_z}"/>
+    <xacro:solid_object
+      name="${name}"
+      x="${x}"
+      y="${y}"
+      z="${z}"
+      roll="${roll}"
+      pitch="${pitch}"
+      yaw="${yaw}"
+      mass="${mass_block}"
+      material="${material}"
+      visible="${visible}"
+    >
+      <xacro:inertia_block
+        mass="${mass_block}"
+        size_x="${size_x}"
+        size_y="${size_y}"
+        size_z="${size_z}"
+      />
+      <box size="${size_x} ${size_y} ${size_z}"/>
+    </xacro:solid_object>
+  </xacro:macro>
+  <!-- Create a solid cylinder of given parameters. -->
+  <xacro:macro
+    name="solid_cylinder"
+    params="
+      name
+      x:=0.0
+      y:=0.0
+      z:=0.0
+      roll:=0.0
+      pitch:=0.0
+      yaw:=0.0
+      radius:=0.5
+      length:=1.0
+      mass:=-1.0
+      material:='Black'
+      visible:=true
+    "
+  >
+    <xacro:property name="mass_cylinder" value="${mass if mass >= 0.0 else DENSITY * length * pi * radius ** 2.0}"/>
+    <xacro:solid_object
+      name="${name}"
+      x="${x}"
+      y="${y}"
+      z="${z}"
+      roll="${roll}"
+      pitch="${pitch}"
+      yaw="${yaw}"
+      mass="${mass_cylinder}"
+      material="${material}"
+      visible="${visible}"
+    >
+      <xacro:inertia_cylinder
+        mass="${mass_cylinder}"
+        radius="${radius}"
+        length="${length}"
+      />
+      <cylinder radius="${radius}" length="${length}"/>
+    </xacro:solid_object>
+  </xacro:macro>
+  <!-- Create a solid sphere of given parameters. -->
+  <xacro:macro
+    name="solid_sphere"
+    params="
+      name
+      x:=0.0
+      y:=0.0
+      z:=0.0
+      roll:=0.0
+      pitch:=0.0
+      yaw:=0.0
+      radius:=0.5
+      mass:=-1.0
+      material:='Black'
+      visible:=true
+    "
+  >
+    <xacro:property name="mass_sphere" value="${mass if mass >= 0.0 else DENSITY * 1.33 * pi * radius ** 2.0}"/>
+    <xacro:solid_object
+      name="${name}"
+      x="${x}"
+      y="${y}"
+      z="${z}"
+      roll="${roll}"
+      pitch="${pitch}"
+      yaw="${yaw}"
+      mass="${mass_sphere}"
+      material="${material}"
+      visible="${visible}"
+    >
+      <xacro:inertia_sphere
+        mass="${mass_sphere}"
+        radius="${radius}"
+      />
+      <sphere radius="${radius}"/>
+    </xacro:solid_object>
+  </xacro:macro>
   <!--
-    Este arquivo assume que o seu domain.xacro (o arquivo que você mostrou)
-    está em: $(find my_robot_description)/urdf/domain.xacro
-    Ajuste o caminho abaixo conforme seu pacote.
+    Create a mesh of given parameters.
+    The filename parameter is a URL, therefore local files should be prepended by
+    "file://", for example:
+    <xacro:solid_mesh name="link_name" filename="file://$(find package_name)/urdf/mesh.stl">
+      ...
+    </xacro:solid_mesh>
   -->
-  <xacro:include filename="$(find my_robot_description)/urdf/domain.xacro"/>
-  <!-- === Parâmetros extraídos do manual Husarion (ROSbot 3) ===
-       - Dimensões (com sensores): 200 x 233 x 197 mm (L x W x H)
-       - Peso (com sensores): 2.84 kg
-       - Standard wheel diameter: ~90 mm (há variações: 85-90 mm em docs)
-       - Wheelbase: 106 mm
-     Fontes: Husarion product/manual. -->
-  <xacro:property name="rosbot_length" value="0.200"/>   <!-- m (200 mm) -->
-  <xacro:property name="rosbot_width"  value="0.233"/>   <!-- m (233 mm) -->
-  <xacro:property name="rosbot_height" value="0.197"/>   <!-- m (197 mm) -->
-  <xacro:property name="rosbot_mass"   value="2.84"/>    <!-- kg (com sensores) -->
-  <xacro:property name="wheel_diameter" value="0.090"/>  <!-- m (90 mm ~ doc: 85-90mm) -->
-  <xacro:property name="wheel_radius"   value="${wheel_diameter / 2.0}"/>
-  <xacro:property name="wheel_width"    value="0.030"/>  <!-- espessura da roda (ajustável) -->
-  <xacro:property name="wheelbase" value="0.106"/>       <!-- m (106 mm) conforme doc -->
-  <!-- track (largura entre eixos das rodas): documento não dá explicitamente.
-       escolhi um valor plausível que cabe na largura total; ajuste se tiver desenho técnico -->
-  <xacro:property name="track" value="0.170"/>           <!-- m (170 mm) - ajuste conforme necessidade -->
-  <!-- chassis thickness (placa de aluminio): -->
-  <xacro:property name="chassis_thickness" value="0.015"/> <!-- 15 mm (valor para visual) -->
-  <!-- localização dos sensores (valores iniciais, ajuste conforme montagem real) -->
-  <xacro:property name="lidar_z" value="${rosbot_height - 0.03}"/>  <!-- perto do topo -->
-  <xacro:property name="camera_z" value="${rosbot_height - 0.06}"/> <!-- um pouco abaixo do LiDAR -->
-  <!-- === Chassis (link base) ===
-       usamos o macro solid_block do domain.xacro para criar o chassi visual/collision -->
-  <xacro:solid_block
-    name="chassis"
-    x="0.0" y="0.0" z="${chassis_thickness/2.0}"  <!-- origin centrado no chão -->
-    size_x="${rosbot_length}"
-    size_y="${rosbot_width}"
-    size_z="${chassis_thickness}"
-    mass="${rosbot_mass * 0.6}"   <!-- parte da massa atribuída ao chassi; resto nas rodas/baterias -->
-    material="DarkGrey"
-    visible="true"
-  />
-  <!-- === Base link (frame) ===
-       criamos um base_link fixo ligado ao chassi (para transform/frame do robô) -->
-  <link name="base_link"/>
-  <xacro:joint_fixed parent="base_link" child="chassis" x="0.0" y="0.0" z="0.0"/>
-  <!-- === Rodas (4) ===
-       posicionamento:
-         x = +- wheelbase/2  (frente/tras)
-         y = +- track/2      (esquerda/direita)
-       usamos solid_cylinder para visual/collision e joint_actuated para tornar as rodas atuadas.
-  -->
-  <!-- roda dianteira esquerda -->
-  <xacro:solid_cylinder
-    name="wheel_fl"
-    x="${wheelbase/2.0}" y="${track/2.0}" z="${wheel_radius}"
-    roll="0" pitch="0" yaw="0"
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