Commit message: correções para atender as características do robot3

File: urdf/domain.xacro (robot description, xacro)
@@ -6,12 +6,12 @@
   Date: 06.11.2025
 -->
-<robot xmlns:xacro="http://www.ros.org/wiki/xacro">
-  <!-- Predefined constants. -->
-  <xacro:property name="M_PI" value="${pi}"/>
-  <xacro:property name="M_PI_2" value="${0.5 * M_PI}"/>
-  <xacro:property name="DEG" value="${M_PI / 180.0}"/>
-  <!-- Default density for computing object mass based on volume. -->
-  <xacro:property name="DENSITY" value="200.0"/>
-  <!-- Pre-defined material colors. -->
+<robot xmlns:xacro="http://www.ros.org/wiki/xacro"> <!-- Definição do namespace xacro -->
+  <!-- Constantes Matemáticas -->
+  <xacro:property name="M_PI" value="${pi}"/> <!-- pi -->
+  <xacro:property name="M_PI_2" value="${0.5 * M_PI}"/> <!-- pi/2 -->
+  <xacro:property name="DEG" value="${M_PI / 180.0}"/> <!-- Grau para radiano -->
+  <!-- Valor padrão de densidade para sólidos (usado quando a massa não é especificada). -->
+  <xacro:property name="DENSITY" value="200.0"/> <!-- kg/m³ -->
+  <!-- Cor dos Materiais -->
   <material name="Black">
     <color rgba="0.0 0.0 0.0 1.0"/>
@@ -29,5 +29,5 @@
     <color rgba="1.0 0.0 0.0 1.0"/>
   </material>
-  <!-- Placeholder inertial tensor. -->
+  <!--  Compute a zero inertial tensor. -->
   <xacro:macro
     name="inertia_none"
@@ -177,86 +177,4 @@
     </xacro:solid_object>
   </xacro:macro>
-  <!-- Create a solid cuboid block of given parameters. -->
-  <xacro:macro
-    name="solid_block_red"
-    params="
-      name
-      x:=0.0
-      y:=0.0
-      z:=0.0
-      roll:=0.0
-      pitch:=0.0
-      yaw:=0.0
-      size_x:=1.0
-      size_y:=1.0
-      size_z:=1.0
-      mass:=-1.0
-      material:='Red'
-      visible:=true
-    "
-  >
-    <xacro:property name="mass_block" value="${mass if mass >= 0.0 else DENSITY * size_x * size_y * size_z}"/>
-    <xacro:solid_object
-      name="${name}"
-      x="${x}"
-      y="${y}"
-      z="${z}"
-      roll="${roll}"
-      pitch="${pitch}"
-      yaw="${yaw}"
-      mass="${mass_block}"
-      material="${material}"
-      visible="${visible}"
-    >
-      <xacro:inertia_block
-        mass="${mass_block}"
-        size_x="${size_x}"
-        size_y="${size_y}"
-        size_z="${size_z}"
-      />
-      <box size="${size_x} ${size_y} ${size_z}"/>
-    </xacro:solid_object>
-  </xacro:macro>
-  <!-- Create a solid cuboid block of given parameters. -->
-  <xacro:macro
-    name="solid_block_black"
-    params="
-      name
-      x:=0.0
-      y:=0.0
-      z:=0.0
-      roll:=0.0
-      pitch:=0.0
-      yaw:=0.0
-      size_x:=1.0
-      size_y:=1.0
-      size_z:=1.0
-      mass:=-1.0
-      material:='Black'
-      visible:=true
-    "
-  >
-    <xacro:property name="mass_block" value="${mass if mass >= 0.0 else DENSITY * size_x * size_y * size_z}"/>
-    <xacro:solid_object
-      name="${name}"
-      x="${x}"
-      y="${y}"
-      z="${z}"
-      roll="${roll}"
-      pitch="${pitch}"
-      yaw="${yaw}"
-      mass="${mass_block}"
-      material="${material}"
-      visible="${visible}"
-    >
-      <xacro:inertia_block
-        mass="${mass_block}"
-        size_x="${size_x}"
-        size_y="${size_y}"
-        size_z="${size_z}"
-      />
-      <box size="${size_x} ${size_y} ${size_z}"/>
-    </xacro:solid_object>
-  </xacro:macro>
   <!-- Create a solid cylinder of given parameters. -->
   <xacro:macro
@@ -311,5 +229,5 @@
       radius:=0.5
       mass:=-1.0
-      material:='Black'
+      material:='Grey'
       visible:=true
     "

File: urdf/gazebo.xacro (robot description, xacro)
@@ -2,5 +2,7 @@
 <!--
   Gazebo extension utilities.
-  Author: Helio Perroni Filho
+  Autor original: Helio Perroni Filho
+  Adaptado por: Vito Rodrigues Franzosi
+  Date: 06.11.2025
 -->
 <robot xmlns:xacro="http://www.ros.org/wiki/xacro">

Commit message: corrigido os erros das rodas do robô e suas dimensões

File: urdf/domain.xacro (robot description, xacro)
@@ -2,16 +2,16 @@
 <!--
   Model primitives.
-  Autor original: Helio Perroni Filho
-  Adaptado por: Vito Rodrigues Franzosi
+  Author: Helio Perroni Filho
+  Adapted by: Vito Rodrigues Franzosi
   Date: 06.11.2025
 -->
-<robot xmlns:xacro="http://www.ros.org/wiki/xacro"> <!-- Definição do namespace xacro -->
-  <!-- Constantes Matemáticas -->
-  <xacro:property name="M_PI" value="${pi}"/> <!-- pi -->
-  <xacro:property name="M_PI_2" value="${0.5 * M_PI}"/> <!-- pi/2 -->
-  <xacro:property name="DEG" value="${M_PI / 180.0}"/> <!-- Grau para radiano -->
-  <!-- Valor padrão de densidade para sólidos (usado quando a massa não é especificada). -->
-  <xacro:property name="DENSITY" value="200.0"/> <!-- kg/m³ -->
-  <!-- Cor dos Materiais -->
+<robot xmlns:xacro="http://www.ros.org/wiki/xacro">
+  <!-- Predefined constants. -->
+  <xacro:property name="M_PI" value="${pi}"/>
+  <xacro:property name="M_PI_2" value="${0.5 * M_PI}"/>
+  <xacro:property name="DEG" value="${M_PI / 180.0}"/>
+  <!-- Default density for computing object mass based on volume. -->
+  <xacro:property name="DENSITY" value="200.0"/>
+  <!-- Pre-defined material colors. -->
   <material name="Black">
     <color rgba="0.0 0.0 0.0 1.0"/>
@@ -29,5 +29,5 @@
     <color rgba="1.0 0.0 0.0 1.0"/>
   </material>
-  <!--  Compute a zero inertial tensor. -->
+  <!-- Placeholder inertial tensor. -->
   <xacro:macro
     name="inertia_none"
@@ -191,5 +191,5 @@
       length:=1.0
       mass:=-1.0
-      material:='Black'
+      material:='Grey'
       visible:=true
     "

File: urdf/gazebo.xacro (robot description, xacro)
@@ -2,6 +2,6 @@
 <!--
   Gazebo extension utilities.
-  Autor original: Helio Perroni Filho
-  Adaptado por: Vito Rodrigues Franzosi
+  Author: Helio Perroni Filho
+  Adapted by: Vito Rodrigues Franzosi
   Date: 06.11.2025
 -->
@@ -108,7 +108,12 @@
       wheel_diameter
       wheel_separation
+      publish_odom:=false
     "
   >
     <gazebo>
+      <plugin name="${name}_joint_states" filename="libgazebo_ros_joint_state_publisher.so">
+        <joint_name>${right_joint}</joint_name>
+        <joint_name>${left_joint}</joint_name>
+      </plugin>
       <plugin name="${name}_controller" filename="libgazebo_ros_diff_drive.so">
         <update_rate>50</update_rate>
@@ -119,12 +124,8 @@
         <max_wheel_torque>20</max_wheel_torque>
         <max_wheel_acceleration>1.0</max_wheel_acceleration>
-        <command_topic>cmd_vel</command_topic>
-        <odometry_topic>odom</odometry_topic>
         <odometry_frame>odom</odometry_frame>
         <robot_base_frame>base_link</robot_base_frame>
-        <publish_odom>true</publish_odom>
-        <publish_odom_tf>true</publish_odom_tf>
-        <publish_wheel_tf>false</publish_wheel_tf>
-        <publish_wheel_joint_state>true</publish_wheel_joint_state>
+        <publish_odom>${publish_odom}</publish_odom>
+        <publish_odom_tf>${publish_odom}</publish_odom_tf>
       </plugin>
     </gazebo>
